Commit message: add ground plane on rviz for ground collision avoidance and change some joint limits

File: kinova_description/urdf/j2n6s300.xacro (robot description, xacro)
@@ -55,5 +55,5 @@
     <xacro:property name="joint_2_origin_xyz" value="0 0.0016 -0.11875" />
     <xacro:property name="joint_2_origin_rpy" value="-${J_PI/2} 0 ${J_PI}" />
-    <xacro:property name="joint_2_lower_limit" value="${47/180*J_PI}" />
+    <xacro:property name="joint_2_lower_limit" value="1.0" />
     <xacro:property name="joint_2_upper_limit" value="${313/180*J_PI}" />
     <xacro:property name="joint_3" value="joint_3" />

File: kinova_description/urdf/j2n6s300_standalone.xacro (robot description, xacro)
@@ -15,4 +15,7 @@
 	xmlns:xacro="http://ros.org/wiki/xacro" name="j2n6s300">
   <xacro:include filename="$(find kinova_description)/urdf/j2n6s300.xacro"/>
+  <xacro:property name="camera_link" value="0.05" />
+  <xacro:property name="height_camera" value="0.157"/>
+  <xacro:property name="axel_offset" value="0.05"/>
   <link name="root">
     <visual>
@@ -39,3 +42,30 @@
   <xacro:property name="robot_root" value="root" />
   <xacro:j2n6s300  base_parent="${robot_root}"/>
+  <!-- for camera sensor -->
+  <joint name="camera_joint" type="fixed">
+    <axis xyz="0 1 0" />
+    <origin xyz="${camera_link} 0 ${height_camera - axel_offset*2}" rpy="0 0 0"/>
+    <parent link="j2n6s300_link_6"/>
+    <child link="camera_link"/>
+  </joint>
+  <link name="camera_link">
+    <collision>
+      <origin xyz="0 0 0" rpy="0 0 0"/>
+      <geometry>
+    <box size="${camera_link} ${camera_link} ${camera_link}"/>
+      </geometry>
+    </collision>
+    <visual>
+      <origin xyz="0 0 0" rpy="0 0 0"/>
+      <geometry>
+    <box size="${camera_link} ${camera_link} ${camera_link}"/>
+      </geometry>
+      <material name="red"/>
+    </visual>
+    <inertial>
+      <mass value="1e-5" />
+      <origin xyz="0 0 0" rpy="0 0 0"/>
+      <inertia ixx="1e-6" ixy="0" ixz="0" iyy="1e-6" iyz="0" izz="1e-6" />
+    </inertial>
+  </link>
 </robot>
