Commit message: clean urdf files

File: jacob_description/urdf/april_box.urdf (robot description, URDF)
Before this commit: robot april_box, 1 links, 0 joints
Links:
- link box: geometry collision mesh filename=package://jacob_description/meshes/april_box.dae; visual mesh filename=package://jacob_description/meshes/april_box.dae

File: jacob_description/urdf/box.urdf (robot description, URDF)
Before this commit: robot tagged_box, 1 links, 0 joints
Links:
- link box: geometry collision mesh filename=package://jacob_description/meshes/tagged_box.dae; visual mesh filename=package://jacob_description/meshes/tagged_box.dae

File: jacob_description/urdf/j2n6s300_standalone.xacro (robot description, xacro)
@@ -54,5 +54,5 @@
       <origin xyz="0 0 0" rpy="0 0 0"/>
       <geometry>
-        <mesh filename="package://kinova_description/meshes/${camera_mesh}.dae"/>
+        <mesh filename="package://jacob_description/meshes/${camera_mesh}.dae"/>
       </geometry>
     </collision>
@@ -60,5 +60,5 @@
       <origin xyz="0 0 0" rpy="1.5707 0 -1.5707"/>
       <geometry>
-        <mesh filename="package://kinova_description/meshes/${camera_mesh}.dae"/>
+        <mesh filename="package://jacob_description/meshes/${camera_mesh}.dae"/>
       </geometry>
       <material name="red"/>

File: jacob_description/urdf/shadded_box.urdf (robot description, URDF)
Before this commit: robot shadded_box, 1 links, 0 joints
Links:
- link box: geometry collision mesh filename=package://jacob_description/meshes/shadded_box.dae; visual mesh filename=package://jacob_description/meshes/shadded_box.dae

File: jacob_description/urdf/simple_box.urdf (robot description, URDF)
Before this commit: robot simple_box, 1 links, 0 joints
Links:
- link box: geometry collision mesh filename=package://jacob_description/meshes/simple_box.dae; visual mesh filename=package://jacob_description/meshes/simple_box.dae

File: jacob_description/urdf/unshadded_box.urdf (robot description, URDF)
Before this commit: robot unshadded_box, 1 links, 0 joints
Links:
- link box: geometry collision mesh filename=package://jacob_description/meshes/unshadded_box.dae; visual mesh filename=package://jacob_description/meshes/unshadded_box.dae

File: jacob_description/urdf/unshaddedtagged_box.urdf (robot description, URDF)
Before this commit: robot unshaddedtagged_box, 1 links, 0 joints
Links:
- link box: geometry collision mesh filename=package://jacob_description/meshes/unshaddedtagged_box.dae; visual mesh filename=package://jacob_description/meshes/unshaddedtagged_box.dae

File: jacob_description/urdf/unshaddedtagged_box2.urdf (robot description, URDF)
Before this commit: robot unshaddedtagged_box2, 1 links, 0 joints
Links:
- link box: geometry collision mesh filename=package://jacob_description/meshes/unshaddedtagged_box2.dae; visual mesh filename=package://jacob_description/meshes/unshaddedtagged_box2.dae
