Commit message: encapsulate jaco urdf

File: jacob_description/urdf/jacob.xacro (robot description, xacro)
@@ -90,5 +90,5 @@
     <xacro:property name="joint_end_effector_origin_xyz" value="0 0 -0.1600" />
     <xacro:property name="joint_end_effector_origin_rpy" value="${J_PI} 0 ${J_PI/2}" />
-    <xacro:macro name="j2s6s300" params="base_parent prefix:=j2s6s300">
+    <xacro:macro name="jacob" params="base_parent prefix:=jacob">
         <xacro:gazebo_config robot_namespace="${prefix}"/>
         <xacro:kinova_armlink link_name="${prefix}_link_base" link_mesh="${link_base_mesh}" mesh_no="${link_base_mesh_no}"/>

File: jacob_description/urdf/jacob_standalone.xacro (robot description, xacro)
@@ -38,4 +38,4 @@
   </joint>
   <xacro:property name="robot_root" value="root" />
-  <xacro:j2s6s300  base_parent="${robot_root}"/>
+  <xacro:jacob  base_parent="${robot_root}"/>
 </robot>
